File: kmSigGenEagle/kmSigGen_Schematics.sch (EAGLE design)
At the start: 42 parts, among them IC1 MEGA8-P

Commit message: Added power supply and update of schematics after review (thx. Zealota & mirekk36 from http://forum.atnel.pl)
Parts:
- removed J2: (no value), con-amp:MTA02-156
- removed R1, R5: 10K, rcl:R-EU_0207/10
- removed R3, R4: 10k, rcl:R-EU_0207/10
- added C12, C13, C14: 100n, capacitor-wima:C2.5/4
- added DCM1, DCM2: ATB-PWR3, _ATNEL:ATB-PWR3
- added L1: 100uH, rcl:L-USIR-2
- C10, C11: value 47uF -> 22uF
- J1: value (none) -> 12V; device con-amp:MTA02-156 -> con-jack:DCJ0303
- SV1: value (none) -> CONNECTOR
Connections:
- removed net ENC_BTN: R20.2
- removed net N$3: DIS1.D0, R1.2
- removed net N$4: DIS1.D1, R5.2
- removed net N$5: DIS1.D2, R3.2
- removed net N$6: DIS1.D3, R4.2
- removed net SCK: SV1.7
- removed net VCC3V: C11.+, J2.2, U$1.VCC
- new net AVCC: C2.2, IC1.AVCC, L1.2
- new net N$7: C12.2, IC1.AREF
- new net VCC3V3: C10.+, C13.2, DCM1.VCC, U$1.VCC
- new net VIN: DCM1.VIN, DCM2.VIN, J1.1
- net ENC_BTTN: now also R20.2
- net GND: now also C12.1, C13.1, C14.1, DCM1.GND, DCM2.GND, J1.2, J1.3; no longer J1.1, J2.1, R1.1, R3.1, R4.1, R5.1
- net SCLK: now also SV1.7
- net VCC: now also C11.+, C14.2, DCM2.VCC, L1.1; no longer C10.+, C2.2, IC1.AVCC, J1.2
Other:
- note added: "POWER SUPPLY"
- note added: "kmSigGen v0.0.4"
- note removed: "TODO: POWER SUPPLY"
- note removed: "kmSigGen v0.0.3"
- moved on the sheet: C1, C10, C11, C2, C5, DEBUG, DIS1, IC1, POWER, R10, R11, R12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
